File: kicad/innerjib7ea-rev-a/innerjib7ea.kicad_sch (KiCad schematic)
At the start: 0 parts

Commit message: feat(hw): rev-A schematic P1 — block diagram
Author the rev-A KiCad 8 schematic top sheet (P1) per the page
breakdown in docs/hw/schematic-page-breakdown.md (Stays PR #35).
P1 is the architectural overview: hierarchical sheet symbols for
the seven sub-pages (P2 ECP5-85F core, P3 DDR3L SO-DIMM, P4 GbE
host link, P5 inter-card connector, P6 USB-UART debug + JTAG, P7
power tree, P8 boot flash) plus annotated bus labels between
them (AXI4 / DDR3L, SGMII, MAST-link, SPI flash, JTAG + UART,
power rails). No real components, no electrical wiring — that
content lands page-by-page in PRs #6c-#6i.

Stub sub-sheets p2..p8 are minimal valid KiCad 8 .kicad_sch
files whose top-level UUIDs match the parent's hierarchical
sheet-symbol UUIDs. Each stub carries an in-page note pointing
the reader at the planning doc section and the placement PR
number that will replace it. This is the structural prerequisite
for the parent's hierarchical sheet symbols to elaborate without
"sheet file not found" ERC errors.

Title block: "POPC_16A rev-A — P1 Block Diagram", date
2026-05-06, rev "A", company "PopSolutions Cooperative", with
comments referencing the planning doc and the project licence
(CERN-OHL-S-2.0 — declared in the directory README per PR #23
since KiCad sexpr cannot embed SPDX inline).

Verification: kicad-cli sch erc --exit-code-violations runs
clean (Found 0 violations) on every .kicad_sch in the project,
including the parent and all seven stubs. KiCad 8.0.9 used
locally via docker (kicad/kicad:8.0); CI re-runs the same check
on ubuntu-24.04 + ppa:kicad/kicad-8.0-releases per
.github/workflows/ci.yml.

Page layout on A3 landscape: ECP5 core in centre (160,110, 60x40
mm); DDR3L / GbE / inter-card stacked on the right column
(270,75 / 270,110 / 270,145); power tree / boot flash / USB-UART
stacked on the left column (50,75 / 50,110 / 50,145); bus labels
positioned in the gaps between blocks.

Out of scope (deferred to subsequent PRs per the planning doc):
real component placement on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
Other:
- added sheet P2_ECP5_Core (p2_ecp5_core.kicad_sch)
- added sheet P3_DDR3L_SODIMM (p3_ddr3l_sodimm.kicad_sch)
- added sheet P4_GbE_HostLink (p4_gbe_hostlink.kicad_sch)
- added sheet P5_InterCard (p5_intercard.kicad_sch)
- added sheet P6_USB_UART_JTAG (p6_usb_uart_jtag.kicad_sch)
- added sheet P7_PowerTree (p7_power_tree.kicad_sch)
- added sheet P8_BootFlash (p8_boot_flash.kicad_sch)
- note added: "AXI4 / DDR3L DQ[15:0], DQS[1:0]_p/n, ADDR[14:0], BA[2:0], CK_p/n, CTRL, ODT, RESET#"
- note added: "Buses shown are inter-sheet contracts; electrical connectivity lands on placement pages P2-P8."
- note added: "Inter-card MAST-link MAST_TX[3:0]_p/n, MAST_RX[3:0]_p/n, sideband + I2C"
- note added: "JTAG + UART TCK, TMS, TDI, TDO, DBG_TXD, DBG_RXD"
- note added: "POPC_16A rev-A — Block Diagram (P1)"
- note added: "Power rails 12V → 3.3V / 2.5V / 1.8V / 1.35V / 1.20V / 1.0V / 0.675V (VTT)"
- note added: "SGMII SGMII_TX_p/n, SGMII_RX_p/n, MDIO, MDC, PHY_INT#"
- note added: "SPI flash bus SPI_CLK, SPI_CS#, SPI_MOSI, SPI_MISO, SPI_WP#, SPI_HOLD#"
- company: (none) -> PopSolutions Cooperative
- title: (none) -> POPC_16A rev-A — P1 Block Diagram
Changed lines of the file:
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@@
 (kicad_sch
 	(version 20231120)
-	(generator "eeschema")
+	(generator "hand_author")
 	(generator_version "8.0")
-	(paper "A4")
-	(symbol_instances)
+	(paper "A3")
+	(title_block
+		(title "POPC_16A rev-A — P1 Block Diagram")
+		(date "2026-05-06")
+		(rev "A")
+		(company "PopSolutions Cooperative")
+		(comment 1 "InnerJib7EA — Lattice ECP5-85F + DDR3L + GbE rev-A")
+		(comment 2 "Hierarchical top sheet (P1). P2-P8 land in subsequent PRs.")
+		(comment 3 "Per docs/hw/schematic-page-breakdown.md (Stays PR #35)")
+		(comment 4 "License: CERN-OHL-S-2.0 (project) — see kicad/innerjib7ea-rev-a/README.md")
+	)
+	(text "POPC_16A rev-A — Block Diagram (P1)"
+		(exclude_from_sim no)
+		(at 210 25 0)
+		(effects
+			(font (size 3.0 3.0) (bold yes))
+			(justify left bottom)
+		)
+	)
+	(text "Buses shown are inter-sheet contracts; electrical connectivity lands on placement pages P2-P8."
+		(exclude_from_sim no)
+		(at 210 35 0)
+		(effects
+			(font (size 1.5 1.5) (italic yes))
+			(justify left bottom)
+		)
+	)
+	(text "AXI4 / DDR3L\nDQ[15:0], DQS[1:0]_p/n,\nADDR[14:0], BA[2:0],\nCK_p/n, CTRL, ODT, RESET#"
+		(exclude_from_sim no)
+		(at 230 95 0)
+		(effects
+			(font (size 1.27 1.27))
+			(justify left bottom)
+		)
+	)
+	(text "SGMII\nSGMII_TX_p/n, SGMII_RX_p/n,\nMDIO, MDC, PHY_INT#"
+		(exclude_from_sim no)
+		(at 230 130 0)
+		(effects
+			(font (size 1.27 1.27))
+			(justify left bottom)
+		)
+	)
+	(text "Inter-card MAST-link\nMAST_TX[3:0]_p/n,\nMAST_RX[3:0]_p/n,\nsideband + I2C"
+		(exclude_from_sim no)
+		(at 230 165 0)
+		(effects
+			(font (size 1.27 1.27))
+			(justify left bottom)
+		)
+	)
+	(text "Power rails\n12V → 3.3V / 2.5V / 1.8V\n/ 1.35V / 1.20V / 1.0V\n/ 0.675V (VTT)"
+		(exclude_from_sim no)
+		(at 130 95 0)
+		(effects
+			(font (size 1.27 1.27))
+			(justify left bottom)
+		)
+	)
+	(text "SPI flash bus\nSPI_CLK, SPI_CS#,\nSPI_MOSI, SPI_MISO,\nSPI_WP#, SPI_HOLD#"
+		(exclude_from_sim no)
+		(at 130 130 0)
+		(effects
+			(font (size 1.27 1.27))
+			(justify left bottom)
+		)
+	)
+	(text "JTAG + UART\nTCK, TMS, TDI, TDO,\nDBG_TXD, DBG_RXD"
+		(exclude_from_sim no)
+		(at 130 165 0)
+		(effects
+			(font (size 1.27 1.27))
+			(justify left bottom)
+		)
+	)
+	(sheet
+		(at 160 110)
+		(size 60 40)
+		(stroke (width 0.5) (type solid))
+		(fill (color 0 0 0 0.0000))
+		(property "Sheetname" "P2_ECP5_Core"
+			(at 160 109.0 0)
+			(effects (font (size 2.0 2.0) (bold yes)) (justify left bottom))
+		)
+		(property "Sheetfile" "p2_ecp5_core.kicad_sch"
+			(at 160 150.5 0)
+			(effects (font (size 1.27 1.27)) (justify left top))
+		)
+		(instances
+			(project "innerjib7ea"
+				(path "/8ac42a0f-deaf-470c-bcc8-9b92c82edf49"
+					(page "2")
+				)
+			)
+		)
+	)
+	(sheet
+		(at 270 75)
+		(size 60 40)
+		(stroke (width 0.3) (type solid))
+		(fill (color 0 0 0 0.0000))
+		(property "Sheetname" "P3_DDR3L_SODIMM"
+			(at 270 74.0 0)
+			(effects (font (size 1.6 1.6) (bold yes)) (justify left bottom))
+		)
+		(property "Sheetfile" "p3_ddr3l_sodimm.kicad_sch"
+			(at 270 115.5 0)
+			(effects (font (size 1.27 1.27)) (justify left top))
+		)
+		(instances
+			(project "innerjib7ea"
+				(path "/8ac42a0f-deaf-470c-bcc8-9b92c82edf49"
+					(page "3")
+				)
+			)
+		)
+	)
+	(sheet
+		(at 270 110)
+		(size 60 40)
+		(stroke (width 0.3) (type solid))
+		(fill (color 0 0 0 0.0000))
+		(property "Sheetname" "P4_GbE_HostLink"
+			(at 270 109.0 0)
+			(effects (font (size 1.6 1.6) (bold yes)) (justify left bottom))
+		)
+		(property "Sheetfile" "p4_gbe_hostlink.kicad_sch"
+			(at 270 150.5 0)
+			(effects (font (size 1.27 1.27)) (justify left top))
+		)
+		(instances
+			(project "innerjib7ea"
+				(path "/8ac42a0f-deaf-470c-bcc8-9b92c82edf49"
+					(page "4")
+				)
+			)
+		)
+	)
+	(sheet
+		(at 270 145)
+		(size 60 40)
+		(stroke (width 0.3) (type solid))
+		(fill (color 0 0 0 0.0000))
+		(property "Sheetname" "P5_InterCard"
+			(at 270 144.0 0)
+			(effects (font (size 1.6 1.6) (bold yes)) (justify left bottom))
+		)
+		(property "Sheetfile" "p5_intercard.kicad_sch"
+			(at 270 185.5 0)
+			(effects (font (size 1.27 1.27)) (justify left top))
+		)
+		(instances
+			(project "innerjib7ea"
+				(path "/8ac42a0f-deaf-470c-bcc8-9b92c82edf49"
+					(page "5")
+				)
+			)
+		)
+	)
+	(sheet
+		(at 50 75)
+		(size 60 40)
+		(stroke (width 0.3) (type solid))
+		(fill (color 0 0 0 0.0000))
+		(property "Sheetname" "P7_PowerTree"
+			(at 50 74.0 0)
+			(effects (font (size 1.6 1.6) (bold yes)) (justify left bottom))
+		)
+		(property "Sheetfile" "p7_power_tree.kicad_sch"
+			(at 50 115.5 0)
+			(effects (font (size 1.27 1.27)) (justify left top))
+		)
+		(instances
+			(project "innerjib7ea"
+				(path "/8ac42a0f-deaf-470c-bcc8-9b92c82edf49"
+					(page "7")
+				)
+			)
+		)
+	)
+	(sheet
+		(at 50 110)
+		(size 60 40)
+		(stroke (width 0.3) (type solid))
+		(fill (color 0 0 0 0.0000))
+		(property "Sheetname" "P8_BootFlash"
+			(at 50 109.0 0)
+			(effects (font (size 1.6 1.6) (bold yes)) (justify left bottom))
+		)
+		(property "Sheetfile" "p8_boot_flash.kicad_sch"
+			(at 50 150.5 0)
+			(effects (font (size 1.27 1.27)) (justify left top))
+		)
+		(instances
+			(project "innerjib7ea"
+				(path "/8ac42a0f-deaf-470c-bcc8-9b92c82edf49"
+					(page "8")
+				)
+			)
+		)
+	)
+	(sheet
+		(at 50 145)
+		(size 60 40)
+		(stroke (width 0.3) (type solid))
+		(fill (color 0 0 0 0.0000))
+		(property "Sheetname" "P6_USB_UART_JTAG"
+			(at 50 144.0 0)
+			(effects (font (size 1.6 1.6) (bold yes)) (justify left bottom))
+		)
+		(property "Sheetfile" "p6_usb_uart_jtag.kicad_sch"
+			(at 50 185.5 0)
+			(effects (font (size 1.27 1.27)) (justify left top))
+		)
+		(instances
+			(project "innerjib7ea"
+				(path "/8ac42a0f-deaf-470c-bcc8-9b92c82edf49"
+					(page "6")
+				)
+			)
+		)
+	)
 	(sheet_instances
-		(path "/"
-			(page "1")
-		)
+		(path "/" (page "1"))
+		(path "/9d93b88c-a1ee-40cd-8803-e89d68343f85" (page "2"))
+		(path "/673f0fd7-1402-4fea-aea3-a0b140daeddb" (page "3"))
+		(path "/8b0158d2-e459-4c49-932e-e09384a66a3d" (page "4"))
+		(path "/860242b0-90fc-4c2e-b114-3b30331e6156" (page "5"))
+		(path "/4ac6ac42-9053-4fb3-8390-45c43313c4b6" (page "6"))
+		(path "/d721d335-5d13-477c-aca4-39777c272ccf" (page "7"))
+		(path "/7f352d9b-1fc1-4a2e-9d42-5a8a1385c71f" (page "8"))
 	)
 )
